Commit message: digital twin rviz and gazebo OK

File: ros2_ws/src/self_balancing_description/urdf/assembly.xacro (robot description, xacro)
@@ -1,7 +1,7 @@
 <?xml version="1.0" ?>
 <robot name="assembly" xmlns:xacro="http://www.ros.org/wiki/xacro">
-<xacro:include filename="$(find assembly_description)/urdf/materials.xacro" />
-<xacro:include filename="$(find assembly_description)/urdf/assembly.trans" />
-<xacro:include filename="$(find assembly_description)/urdf/assembly.gazebo" />
+<xacro:include filename="$(find self_balancing_description)/urdf/materials.xacro" />
+<xacro:include filename="$(find self_balancing_description)/urdf/assembly.trans" />
+<xacro:include filename="$(find self_balancing_description)/urdf/assembly.gazebo" />
 <link name="base_link">
   <inertial>
@@ -13,5 +13,5 @@
     <origin xyz="0 0 0" rpy="0 0 0"/>
     <geometry>
-      <mesh filename="file://$(find assembly_description)/meshes/base_link.stl" scale="0.001 0.001 0.001"/>
+      <mesh filename="file://$(find self_balancing_description)/meshes/base_link.stl" scale="0.001 0.001 0.001"/>
     </geometry>
     <material name="silver"/>
@@ -20,5 +20,5 @@
     <origin xyz="0 0 0" rpy="0 0 0"/>
     <geometry>
-      <mesh filename="file://$(find assembly_description)/meshes/base_link.stl" scale="0.001 0.001 0.001"/>
+      <mesh filename="file://$(find self_balancing_description)/meshes/base_link.stl" scale="0.001 0.001 0.001"/>
     </geometry>
   </collision>
@@ -33,5 +33,5 @@
     <origin xyz="-0.0 -0.1 -0.0" rpy="0 0 0"/>
     <geometry>
-      <mesh filename="file://$(find assembly_description)/meshes/Aluminium_20x20_250_back_1.stl" scale="0.001 0.001 0.001"/>
+      <mesh filename="file://$(find self_balancing_description)/meshes/Aluminium_20x20_250_back_1.stl" scale="0.001 0.001 0.001"/>
     </geometry>
     <material name="silver"/>
@@ -40,5 +40,5 @@
     <origin xyz="-0.0 -0.1 -0.0" rpy="0 0 0"/>
     <geometry>
-      <mesh filename="file://$(find assembly_description)/meshes/Aluminium_20x20_250_back_1.stl" scale="0.001 0.001 0.001"/>
+      <mesh filename="file://$(find self_balancing_description)/meshes/Aluminium_20x20_250_back_1.stl" scale="0.001 0.001 0.001"/>
     </geometry>
   </collision>
@@ -53,5 +53,5 @@
     <origin xyz="-0.0 -0.0 -0.0" rpy="0 0 0"/>
     <geometry>
-      <mesh filename="file://$(find assembly_description)/meshes/Battery_1.stl" scale="0.001 0.001 0.001"/>
+      <mesh filename="file://$(find self_balancing_description)/meshes/Battery_1.stl" scale="0.001 0.001 0.001"/>
     </geometry>
     <material name="silver"/>
@@ -60,5 +60,5 @@
     <origin xyz="-0.0 -0.0 -0.0" rpy="0 0 0"/>
     <geometry>
-      <mesh filename="file://$(find assembly_description)/meshes/Battery_1.stl" scale="0.001 0.001 0.001"/>
+      <mesh filename="file://$(find self_balancing_description)/meshes/Battery_1.stl" scale="0.001 0.001 0.001"/>
     </geometry>
   </collision>
@@ -73,5 +73,5 @@
     <origin xyz="-0.1278 -0.0804 0.135" rpy="0 0 0"/>
     <geometry>
-      <mesh filename="file://$(find assembly_description)/meshes/Aluminium_20x40_160_left_1.stl" scale="0.001 0.001 0.001"/>
+      <mesh filename="file://$(find self_balancing_description)/meshes/Aluminium_20x40_160_left_1.stl" scale="0.001 0.001 0.001"/>
     </geometry>
     <material name="silver"/>
@@ -80,5 +80,5 @@
     <origin xyz="-0.1278 -0.0804 0.135" rpy="0 0 0"/>
     <geometry>
-      <mesh filename="file://$(find assembly_description)/meshes/Aluminium_20x40_160_left_1.stl" scale="0.001 0.001 0.001"/>
+      <mesh filename="file://$(find self_balancing_description)/meshes/Aluminium_20x40_160_left_1.stl" scale="0.001 0.001 0.001"/>
     </geometry>
   </collision>
@@ -93,5 +93,5 @@
     <origin xyz="-0.1278 -0.0804 -0.115" rpy="0 0 0"/>
     <geometry>
-      <mesh filename="file://$(find assembly_description)/meshes/Aluminium_20x40_160_right_1.stl" scale="0.001 0.001 0.001"/>
+      <mesh filename="file://$(find self_balancing_description)/meshes/Aluminium_20x40_160_right_1.stl" scale="0.001 0.001 0.001"/>
     </geometry>
     <material name="silver"/>
@@ -100,5 +100,5 @@
     <origin xyz="-0.1278 -0.0804 -0.115" rpy="0 0 0"/>
     <geometry>
-      <mesh filename="file://$(find assembly_description)/meshes/Aluminium_20x40_160_right_1.stl" scale="0.001 0.001 0.001"/>
+      <mesh filename="file://$(find self_balancing_description)/meshes/Aluminium_20x40_160_right_1.stl" scale="0.001 0.001 0.001"/>
     </geometry>
   </collision>
@@ -113,5 +113,5 @@
     <origin xyz="-0.2 0.0198 -0.0023" rpy="0 0 0"/>
     <geometry>
-      <mesh filename="file://$(find assembly_description)/meshes/Shaft_Collar_16mm_left1_1.stl" scale="0.001 0.001 0.001"/>
+      <mesh filename="file://$(find self_balancing_description)/meshes/Shaft_Collar_16mm_left1_1.stl" scale="0.001 0.001 0.001"/>
     </geometry>
     <material name="silver"/>
@@ -120,5 +120,5 @@
     <origin xyz="-0.2 0.0198 -0.0023" rpy="0 0 0"/>
     <geometry>
-      <mesh filename="file://$(find assembly_description)/meshes/Shaft_Collar_16mm_left1_1.stl" scale="0.001 0.001 0.001"/>
+      <mesh filename="file://$(find self_balancing_description)/meshes/Shaft_Collar_16mm_left1_1.stl" scale="0.001 0.001 0.001"/>
     </geometry>
   </collision>
@@ -133,5 +133,5 @@
     <origin xyz="0.23 -0.0033 0.0898" rpy="0 0 0"/>
     <geometry>
-      <mesh filename="file://$(find assembly_description)/meshes/Aluminium_20x20_250_front_1.stl" scale="0.001 0.001 0.001"/>
+      <mesh filename="file://$(find self_balancing_description)/meshes/Aluminium_20x20_250_front_1.stl" scale="0.001 0.001 0.001"/>
     </geometry>
     <material name="silver"/>
@@ -140,5 +140,5 @@
     <origin xyz="0.23 -0.0033 0.0898" rpy="0 0 0"/>
     <geometry>
-      <mesh filename="file://$(find assembly_description)/meshes/Aluminium_20x20_250_front_1.stl" scale="0.001 0.001 0.001"/>
+      <mesh filename="file://$(find self_balancing_description)/meshes/Aluminium_20x20_250_front_1.stl" scale="0.001 0.001 0.001"/>
     </geometry>
   </collision>
@@ -153,5 +153,5 @@
     <origin xyz="0.22 -0.0002 -0.0027" rpy="0 0 0"/>
     <geometry>
-      <mesh filename="file://$(find assembly_description)/meshes/Shaft_Collar_16mm_right2_1.stl" scale="0.001 0.001 0.001"/>
+      <mesh filename="file://$(find self_balancing_description)/meshes/Shaft_Collar_16mm_right2_1.stl" scale="0.001 0.001 0.001"/>
     </geometry>
     <material name="silver"/>
@@ -160,5 +160,5 @@
     <origin xyz="0.22 -0.0002 -0.0027" rpy="0 0 0"/>
     <geometry>
-      <mesh filename="file://$(find assembly_description)/meshes/Shaft_Collar_16mm_right2_1.stl" scale="0.001 0.001 0.001"/>
+      <mesh filename="file://$(find self_balancing_description)/meshes/Shaft_Collar_16mm_right2_1.stl" scale="0.001 0.001 0.001"/>
     </geometry>
   </collision>
@@ -173,5 +173,5 @@
     <origin xyz="-0.22 0.0198 0.0227" rpy="0 0 0"/>
     <geometry>
-      <mesh filename="file://$(find assembly_description)/meshes/Shaft_Collar_16mm_left2_1.stl" scale="0.001 0.001 0.001"/>
+      <mesh filename="file://$(find self_balancing_description)/meshes/Shaft_Collar_16mm_left2_1.stl" scale="0.001 0.001 0.001"/>
     </geometry>
     <material name="silver"/>
@@ -180,5 +180,5 @@
     <origin xyz="-0.22 0.0198 0.0227" rpy="0 0 0"/>
     <geometry>
-      <mesh filename="file://$(find assembly_description)/meshes/Shaft_Collar_16mm_left2_1.stl" scale="0.001 0.001 0.001"/>
+      <mesh filename="file://$(find self_balancing_description)/meshes/Shaft_Collar_16mm_left2_1.stl" scale="0.001 0.001 0.001"/>
     </geometry>
   </collision>
@@ -193,5 +193,5 @@
     <origin xyz="0.2 -0.0002 -0.0027" rpy="0 0 0"/>
     <geometry>
-      <mesh filename="file://$(find assembly_description)/meshes/Shaft_Collar_16mm_right1_1.stl" scale="0.001 0.001 0.001"/>
+      <mesh filename="file://$(find self_balancing_description)/meshes/Shaft_Collar_16mm_right1_1.stl" scale="0.001 0.001 0.001"/>
     </geometry>
     <material name="silver"/>
@@ -200,5 +200,5 @@
     <origin xyz="0.2 -0.0002 -0.0027" rpy="0 0 0"/>
     <geometry>
-      <mesh filename="file://$(find assembly_description)/meshes/Shaft_Collar_16mm_right1_1.stl" scale="0.001 0.001 0.001"/>
+      <mesh filename="file://$(find self_balancing_description)/meshes/Shaft_Collar_16mm_right1_1.stl" scale="0.001 0.001 0.001"/>
     </geometry>
   </collision>
@@ -213,5 +213,5 @@
     <origin xyz="-0.125 -0.083 -0.0" rpy="0 0 0"/>
     <geometry>
-      <mesh filename="file://$(find assembly_description)/meshes/Aluminium_20x20_100_back_left_1.stl" scale="0.001 0.001 0.001"/>
+      <mesh filename="file://$(find self_balancing_description)/meshes/Aluminium_20x20_100_back_left_1.stl" scale="0.001 0.001 0.001"/>
     </geometry>
     <material name="silver"/>
@@ -220,5 +220,5 @@
     <origin xyz="-0.125 -0.083 -0.0" rpy="0 0 0"/>
     <geometry>
-      <mesh filename="file://$(find assembly_description)/meshes/Aluminium_20x20_100_back_left_1.stl" scale="0.001 0.001 0.001"/>
+      <mesh filename="file://$(find self_balancing_description)/meshes/Aluminium_20x20_100_back_left_1.stl" scale="0.001 0.001 0.001"/>
     </geometry>
   </collision>
@@ -233,5 +233,5 @@
     <origin xyz="0.125 -0.0974 0.0" rpy="0 0 0"/>
     <geometry>
-      <mesh filename="file://$(find assembly_description)/meshes/Aluminium_20x20_100_back_right_1.stl" scale="0.001 0.001 0.001"/>
+      <mesh filename="file://$(find self_balancing_description)/meshes/Aluminium_20x20_100_back_right_1.stl" scale="0.001 0.001 0.001"/>
     </geometry>
     <material name="silver"/>
@@ -240,5 +240,5 @@
     <origin xyz="0.125 -0.0974 0.0" rpy="0 0 0"/>
     <geometry>
-      <mesh filename="file://$(find assembly_description)/meshes/Aluminium_20x20_100_back_right_1.stl" scale="0.001 0.001 0.001"/>
+      <mesh filename="file://$(find self_balancing_description)/meshes/Aluminium_20x20_100_back_right_1.stl" scale="0.001 0.001 0.001"/>
     </geometry>
   </collision>
@@ -253,5 +253,5 @@
     <origin xyz="0.125 0.0826 0.0" rpy="0 0 0"/>
     <geometry>
-      <mesh filename="file://$(find assembly_description)/meshes/Aluminium_20x20_100_front_right_1.stl" scale="0.001 0.001 0.001"/>
+      <mesh filename="file://$(find self_balancing_description)/meshes/Aluminium_20x20_100_front_right_1.stl" scale="0.001 0.001 0.001"/>
     </geometry>
     <material name="silver"/>
@@ -260,5 +260,5 @@
     <origin xyz="0.125 0.0826 0.0" rpy="0 0 0"/>
     <geometry>
-      <mesh filename="file://$(find assembly_description)/meshes/Aluminium_20x20_100_front_right_1.stl" scale="0.001 0.001 0.001"/>
+      <mesh filename="file://$(find self_balancing_description)/meshes/Aluminium_20x20_100_front_right_1.stl" scale="0.001 0.001 0.001"/>
     </geometry>
   </collision>
@@ -273,5 +273,5 @@
     <origin xyz="-0.125 0.097 -0.0" rpy="0 0 0"/>
     <geometry>
-      <mesh filename="file://$(find assembly_description)/meshes/Aluminium_20x20_100_front_left_1.stl" scale="0.001 0.001 0.001"/>
+      <mesh filename="file://$(find self_balancing_description)/meshes/Aluminium_20x20_100_front_left_1.stl" scale="0.001 0.001 0.001"/>
     </geometry>
     <material name="silver"/>
@@ -280,5 +280,5 @@
     <origin xyz="-0.125 0.097 -0.0" rpy="0 0 0"/>
     <geometry>
-      <mesh filename="file://$(find assembly_description)/meshes/Aluminium_20x20_100_front_left_1.stl" scale="0.001 0.001 0.001"/>
+      <mesh filename="file://$(find self_balancing_description)/meshes/Aluminium_20x20_100_front_left_1.stl" scale="0.001 0.001 0.001"/>
     </geometry>
   </collision>
@@ -293,5 +293,5 @@
     <origin xyz="0.125 0.097 -0.1" rpy="0 0 0"/>
     <geometry>
-      <mesh filename="file://$(find assembly_description)/meshes/Aluminium_20x20_250_top_front_1.stl" scale="0.001 0.001 0.001"/>
+      <mesh filename="file://$(find self_balancing_description)/meshes/Aluminium_20x20_250_top_front_1.stl" scale="0.001 0.001 0.001"/>
     </geometry>
     <material name="silver"/>
@@ -300,5 +300,5 @@
     <origin xyz="0.125 0.097 -0.1" rpy="0 0 0"/>
     <geometry>
-      <mesh filename="file://$(find assembly_description)/meshes/Aluminium_20x20_250_top_front_1.stl" scale="0.001 0.001 0.001"/>
+      <mesh filename="file://$(find self_balancing_description)/meshes/Aluminium_20x20_250_top_front_1.stl" scale="0.001 0.001 0.001"/>
     </geometry>
   </collision>
@@ -313,5 +313,5 @@
     <origin xyz="0.125 -0.083 -0.1" rpy="0 0 0"/>
     <geometry>
-      <mesh filename="file://$(find assembly_description)/meshes/Aluminium_20x20_250_top_back_1.stl" scale="0.001 0.001 0.001"/>
+      <mesh filename="file://$(find self_balancing_description)/meshes/Aluminium_20x20_250_top_back_1.stl" scale="0.001 0.001 0.001"/>
     </geometry>
     <material name="silver"/>
@@ -320,5 +320,5 @@
     <origin xyz="0.125 -0.083 -0.1" rpy="0 0 0"/>
     <geometry>
-      <mesh filename="file://$(find assembly_description)/meshes/Aluminium_20x20_250_top_back_1.stl" scale="0.001 0.001 0.001"/>
+      <mesh filename="file://$(find self_balancing_description)/meshes/Aluminium_20x20_250_top_back_1.stl" scale="0.001 0.001 0.001"/>
     </geometry>
   </collision>
@@ -333,5 +333,5 @@
     <origin xyz="0.125 0.0798 -0.1172" rpy="0 0 0"/>
     <geometry>
-      <mesh filename="file://$(find assembly_description)/meshes/Aluminium_20x20_160_right_1.stl" scale="0.001 0.001 0.001"/>
+      <mesh filename="file://$(find self_balancing_description)/meshes/Aluminium_20x20_160_right_1.stl" scale="0.001 0.001 0.001"/>
     </geometry>
     <material name="silver"/>
@@ -340,5 +340,5 @@
     <origin xyz="0.125 0.0798 -0.1172" rpy="0 0 0"/>
     <geometry>
-      <mesh filename="file://$(find assembly_description)/meshes/Aluminium_20x20_160_right_1.stl" scale="0.001 0.001 0.001"/>
+      <mesh filename="file://$(find self_balancing_description)/meshes/Aluminium_20x20_160_right_1.stl" scale="0.001 0.001 0.001"/>
     </geometry>
   </collision>
@@ -353,5 +353,5 @@
     <origin xyz="-0.125 0.0798 -0.1172" rpy="0 0 0"/>
     <geometry>
-      <mesh filename="file://$(find assembly_description)/meshes/Aluminium_20x20_160_left_1.stl" scale="0.001 0.001 0.001"/>
+      <mesh filename="file://$(find self_balancing_description)/meshes/Aluminium_20x20_160_left_1.stl" scale="0.001 0.001 0.001"/>
     </geometry>
     <material name="silver"/>
@@ -360,5 +360,5 @@
     <origin xyz="-0.125 0.0798 -0.1172" rpy="0 0 0"/>
     <geometry>
-      <mesh filename="file://$(find assembly_description)/meshes/Aluminium_20x20_160_left_1.stl" scale="0.001 0.001 0.001"/>
+      <mesh filename="file://$(find self_balancing_description)/meshes/Aluminium_20x20_160_left_1.stl" scale="0.001 0.001 0.001"/>
     </geometry>
   </collision>
@@ -373,5 +373,5 @@
     <origin xyz="-0.2299 -0.0402 -0.1998" rpy="0 0 0"/>
     <geometry>
-      <mesh filename="file://$(find assembly_description)/meshes/encoder_holding_left_1.stl" scale="0.001 0.001 0.001"/>
+      <mesh filename="file://$(find self_balancing_description)/meshes/encoder_holding_left_1.stl" scale="0.001 0.001 0.001"/>
     </geometry>
     <material name="silver"/>
@@ -380,5 +380,5 @@
     <origin xyz="-0.2299 -0.0402 -0.1998" rpy="0 0 0"/>
     <geometry>
-      <mesh filename="file://$(find assembly_description)/meshes/encoder_holding_left_1.stl" scale="0.001 0.001 0.001"/>
+      <mesh filename="file://$(find self_balancing_description)/meshes/encoder_holding_left_1.stl" scale="0.001 0.001 0.001"/>
     </geometry>
   </collision>
@@ -393,5 +393,5 @@
     <origin xyz="0.2301 -0.0402 -0.1998" rpy="0 0 0"/>
     <geometry>
-      <mesh filename="file://$(find assembly_description)/meshes/encoder_holding_right_1.stl" scale="0.001 0.001 0.001"/>
+      <mesh filename="file://$(find self_balancing_description)/meshes/encoder_holding_right_1.stl" scale="0.001 0.001 0.001"/>
     </geometry>
     <material name="silver"/>
@@ -400,5 +400,5 @@
     <origin xyz="0.2301 -0.0402 -0.1998" rpy="0 0 0"/>
     <geometry>
-      <mesh filename="file://$(find assembly_description)/meshes/encoder_holding_right_1.stl" scale="0.001 0.001 0.001"/>
+      <mesh filename="file://$(find self_balancing_description)/meshes/encoder_holding_right_1.stl" scale="0.001 0.001 0.001"/>
     </geometry>
   </collision>
@@ -413,5 +413,5 @@
     <origin xyz="-0.1124 0.0073 -0.00701" rpy="0 0 0"/>
     <geometry>
-      <mesh filename="file://$(find assembly_description)/meshes/E6B2_CWZ6C_left_1.stl" scale="0.001 0.001 0.001"/>
+      <mesh filename="file://$(find self_balancing_description)/meshes/E6B2_CWZ6C_left_1.stl" scale="0.001 0.001 0.001"/>
     </geometry>
     <material name="silver"/>
@@ -420,5 +420,5 @@
     <origin xyz="-0.1124 0.0073 -0.00701" rpy="0 0 0"/>
     <geometry>
-      <mesh filename="file://$(find assembly_description)/meshes/E6B2_CWZ6C_left_1.stl" scale="0.001 0.001 0.001"/>
+      <mesh filename="file://$(find self_balancing_description)/meshes/E6B2_CWZ6C_left_1.stl" scale="0.001 0.001 0.001"/>
     </geometry>
   </collision>
@@ -433,5 +433,5 @@
     <origin xyz="0.1126 0.0148 -0.02" rpy="0 0 0"/>
     <geometry>
-      <mesh filename="file://$(find assembly_description)/meshes/E6B2_CWZ6C_right_1.stl" scale="0.001 0.001 0.001"/>
+      <mesh filename="file://$(find self_balancing_description)/meshes/E6B2_CWZ6C_right_1.stl" scale="0.001 0.001 0.001"/>
     </geometry>
     <material name="silver"/>
@@ -440,5 +440,5 @@
     <origin xyz="0.1126 0.0148 -0.02" rpy="0 0 0"/>
     <geometry>
-      <mesh filename="file://$(find assembly_description)/meshes/E6B2_CWZ6C_right_1.stl" scale="0.001 0.001 0.001"/>
+      <mesh filename="file://$(find self_balancing_description)/meshes/E6B2_CWZ6C_right_1.stl" scale="0.001 0.001 0.001"/>
     </geometry>
   </collision>
@@ -453,5 +453,5 @@
     <origin xyz="0.085 -0.0002 0.0196" rpy="0 0 0"/>
     <geometry>
-      <mesh filename="file://$(find assembly_description)/meshes/shaft_right_1.stl" scale="0.001 0.001 0.001"/>
+      <mesh filename="file://$(find self_balancing_description)/meshes/shaft_right_1.stl" scale="0.001 0.001 0.001"/>
     </geometry>
     <material name="silver"/>
@@ -460,5 +460,5 @@
     <origin xyz="0.085 -0.0002 0.0196" rpy="0 0 0"/>
     <geometry>
-      <mesh filename="file://$(find assembly_description)/meshes/shaft_right_1.stl" scale="0.001 0.001 0.001"/>
+      <mesh filename="file://$(find self_balancing_description)/meshes/shaft_right_1.stl" scale="0.001 0.001 0.001"/>
     </geometry>
   </collision>
@@ -473,5 +473,5 @@
     <origin xyz="-0.085 -0.0002 0.0196" rpy="0 0 0"/>
     <geometry>
-      <mesh filename="file://$(find assembly_description)/meshes/shaft_left_1.stl" scale="0.001 0.001 0.001"/>
+      <mesh filename="file://$(find self_balancing_description)/meshes/shaft_left_1.stl" scale="0.001 0.001 0.001"/>
     </geometry>
     <material name="silver"/>
@@ -480,5 +480,5 @@
     <origin xyz="-0.085 -0.0002 0.0196" rpy="0 0 0"/>
     <geometry>
-      <mesh filename="file://$(find assembly_description)/meshes/shaft_left_1.stl" scale="0.001 0.001 0.001"/>
+      <mesh filename="file://$(find self_balancing_description)/meshes/shaft_left_1.stl" scale="0.001 0.001 0.001"/>
     </geometry>
   </collision>
@@ -493,5 +493,5 @@
     <origin xyz="0.1326 -0.0002 0.0251" rpy="0 0 0"/>
     <geometry>
-      <mesh filename="file://$(find assembly_description)/meshes/wheel_right_1.stl" scale="0.001 0.001 0.001"/>
+      <mesh filename="file://$(find self_balancing_description)/meshes/wheel_right_1.stl" scale="0.001 0.001 0.001"/>
     </geometry>
     <material name="silver"/>
@@ -500,5 +500,5 @@
     <origin xyz="0.1326 -0.0002 0.0251" rpy="0 0 0"/>
     <geometry>
-      <mesh filename="file://$(find assembly_description)/meshes/wheel_right_1.stl" scale="0.001 0.001 0.001"/>
+      <mesh filename="file://$(find self_balancing_description)/meshes/wheel_right_1.stl" scale="0.001 0.001 0.001"/>
     </geometry>
   </collision>
@@ -513,5 +513,5 @@
     <origin xyz="-0.1326 -0.0002 0.0251" rpy="0 0 0"/>
     <geometry>
-      <mesh filename="file://$(find assembly_description)/meshes/wheel_left_1.stl" scale="0.001 0.001 0.001"/>
+      <mesh filename="file://$(find self_balancing_description)/meshes/wheel_left_1.stl" scale="0.001 0.001 0.001"/>
     </geometry>
     <material name="silver"/>
@@ -520,5 +520,5 @@
     <origin xyz="-0.1326 -0.0002 0.0251" rpy="0 0 0"/>
     <geometry>
-      <mesh filename="file://$(find assembly_description)/meshes/wheel_left_1.stl" scale="0.001 0.001 0.001"/>
+      <mesh filename="file://$(find self_balancing_description)/meshes/wheel_left_1.stl" scale="0.001 0.001 0.001"/>
     </geometry>
   </collision>
